Commit message: fix urdf ur rbtq integration

File: ur5_robotiq_description/urdf/ur_with_2f85_base.urdf.xacro (robot description, xacro)
@@ -28,5 +28,5 @@
       safety_k_position="20"
       force_abs_paths="true">
-    <origin xyz="0 0 0" rpy="0 0 0"/>
+    <origin xyz="0 0 0" rpy="0 0 1.5707"/>
   </xacro:ur_robot>
   <!-- ========================================================= -->

File: ur5_robotiq_description/urdf/ur_with_2f85_moveit.urdf.xacro (robot description, xacro)
@@ -3,5 +3,5 @@
   <!-- Include ONLY the base robot -->
 <xacro:include
-    filename="$(find ur5_robotiq_description)/urdf/ur_with_gripper_base.urdf.xacro"/>
+    filename="$(find ur5_robotiq_description)/urdf/ur_with_2f85_base.urdf.xacro"/>
 <link name="world"/>
 <joint name="world_to_base" type="fixed">

File: ur5_robotiq_description/urdf/ur_with_2f85_sim.urdf.xacro (robot description, xacro)
@@ -1,3 +1,2 @@
-```xml
 <?xml version="1.0"?>
 <robot xmlns:xacro="http://www.ros.org/wiki/xacro" name="$(arg name)">
@@ -14,41 +13,22 @@
   <!-- ========================================================= -->
   <xacro:include
-      filename="$(find ur5_robotiq_description)/urdf/ur_with_gripper_base.urdf.xacro"/>
+      filename="$(find ur5_robotiq_description)/urdf/ur_with_2f85_base.urdf.xacro"/>
   <!-- ========================================================= -->
   <!-- World and ground plane                                    -->
   <!-- ========================================================= -->
-  <link name="world"/>
-  <link name="ground_plane">
-    <visual>
-      <geometry>
-        <box size="5 5 0.02"/>
-      </geometry>
-      <material name="ground_white">
-        <color rgba="1 1 1 0.5"/>
-      </material>
-    </visual>
-    <collision>
-      <geometry>
-        <box size="5 5 0.02"/>
-      </geometry>
-    </collision>
-  </link>
-  <joint name="ground_plane_joint" type="fixed">
-    <parent link="world"/>
-    <child link="ground_plane"/>
-    <origin xyz="0 0 -0.01" rpy="0 0 0"/>
-  </joint>
-  <!-- Mount the robot base to the world. -->
-  <joint name="base_mount" type="fixed">
-    <parent link="world"/>
-    <child link="base_link_parent"/>
-    <origin xyz="0 0 0" rpy="0 0 0"/>
-  </joint>
+  <!-- World reference frame -->
+<link name="world"/>
+<!-- Mount the robot base to the world -->
+<joint name="base_mount" type="fixed">
+  <parent link="world"/>
+  <child link="base_link_parent"/>
+  <origin xyz="0 0 0" rpy="0 0 0"/>
+</joint>
   <!-- ========================================================= -->
   <!-- Gazebo ros2_control plugin                                -->
   <!-- ========================================================= -->
-  <gazebo>
+  <!-- <gazebo>
     <plugin
-        filename="libgz_ros2_control-system.so"
+        filename="gz_ros2_control-system.so"
         name="gz_ros2_control::GazeboSimROS2ControlPlugin">
       <parameters>$(arg simulation_controllers)</parameters>
@@ -56,4 +36,11 @@
         <namespace>$(arg ros_namespace)</namespace>
       </ros>
+    </plugin>
+  </gazebo> -->
+  <gazebo>
+    <plugin
+        filename="gz_ros2_control-system"
+        name="gz_ros2_control::GazeboSimROS2ControlPlugin">
+      <parameters>$(arg simulation_controllers)</parameters>
     </plugin>
   </gazebo>
@@ -65,7 +52,7 @@
       <plugin>gz_ros2_control/GazeboSimSystem</plugin>
     </hardware>
-    <!-- ------------------------------------------------------- -->
+    <!-- ========================================================= -->
     <!-- UR5 arm joints                                         -->
-    <!-- ------------------------------------------------------- -->
+    <!-- ========================================================= -->
     <joint name="shoulder_pan_joint">
       <command_interface name="position"/>
@@ -98,25 +85,46 @@
       <state_interface name="velocity"/>
     </joint>
-    <!-- ------------------------------------------------------- -->
+    <!-- ========================================================= -->
     <!-- Robotiq 2F-85 actuated joint                            -->
-    <!-- ------------------------------------------------------- -->
+    <!-- ========================================================= -->
+   <!-- Robotiq 2F-85: actuated joint -->
     <joint name="robotiq_85_left_knuckle_joint">
       <command_interface name="position"/>
       <state_interface name="position">
-        <param name="initial_value">0.7929</param>
+        <param name="initial_value">0.0</param>
       </state_interface>
       <state_interface name="velocity"/>
     </joint>
-    <!-- ------------------------------------------------------- -->
+    <!-- Mimic joints: state interfaces only; no independent commands -->
+    <joint name="robotiq_85_right_knuckle_joint">
+      <state_interface name="position"/>
+      <state_interface name="velocity"/>
+    </joint>
+    <joint name="robotiq_85_left_inner_knuckle_joint">
+      <state_interface name="position"/>
+      <state_interface name="velocity"/>
+    </joint>
+    <joint name="robotiq_85_right_inner_knuckle_joint">
+      <state_interface name="position"/>
+      <state_interface name="velocity"/>
+    </joint>
+    <joint name="robotiq_85_left_finger_tip_joint">
+      <state_interface name="position"/>
+      <state_interface name="velocity"/>
+    </joint>
+    <joint name="robotiq_85_right_finger_tip_joint">
+      <state_interface name="position"/>
+      <state_interface name="velocity"/>
+    </joint>
+    <!-- ========================================================= -->
     <!-- Robotiq mimic joints                                    -->
     <!-- Gazebo is responsible for their mimic behavior.         -->
     <!-- Do not expose independent command interfaces.           -->
-    <!-- ------------------------------------------------------- -->
-    <joint name="robotiq_85_right_knuckle_joint"/>
+    <!-- ========================================================= -->
+    <!-- <joint name="robotiq_85_right_knuckle_joint"/>
     <joint name="robotiq_85_left_inner_knuckle_joint"/>
     <joint name="robotiq_85_right_inner_knuckle_joint"/>
     <joint name="robotiq_85_left_finger_tip_joint"/>
-    <joint name="robotiq_85_right_finger_tip_joint"/>
+    <joint name="robotiq_85_right_finger_tip_joint"/> -->
   </ros2_control>
 </robot>
-```
